File: THW/Eagle/THW_Design/v1.2.0.sch (EAGLE design)
At the start: 41 parts, among them U1 ADA4091-2ARZ-RL

Commit message: commit
Parts:
- removed C1: 0805YC103J4T2A, 0805YC103J4T2A:0805YC103J4T2A
- removed R1, R2, R3: (no value), resistor:R-US_M0805
- removed U1: ADA4091-2ARZ-RL, ADA4091-2ARZ-RL:ADA4091-2ARZ-RL
Connections:
- removed net GND: C1.C2, POWER.6, R3.2, U1.INA+, U1.V-, WB_SENS2.8
- removed net LONG_HW+: U1.INA-
- removed net LONG_HW_SENS-: LONG_HW-.P$1, TP28.TP, WB_SENS1.2
- removed net N$2: R1.1, U1.INB+
- removed net N$4: R2.2, R3.1, U1.INB-
- removed net OPAMP_OUTPUT: R2.1, U1.OUTB, WB_SENS2.7
- removed net SHORT_HW_SENS+: SHORT_HW+.P$2, TP26.TP, WB_SENS1.8
- removed net SHORT_HW_SENS-: LONG_HW+.P$2, SHORT_HW-.P$1, TP25.TP, TP27.TP, WB_SENS1.1, WB_SENS1.5, WB_SENS1.7
- removed net SUMMING_OP_AMP: R1.2, R4.1, R7.2, WB_SENS1.6, WB_SENS2.4, WB_SENS2.5
- removed net VSS: C1.C1, POWER.5, U1.V+
- new net NODE_B: R4.1, R7.2, WB_SENS1.7, WB_SENS2.4, WB_SENS2.6
- net SHORT_HW+: now also SHORT_HW+.P$2, TP26.TP, WB_SENS1.2, WB_SENS2.5, WB_SENS2.8; no longer WB_SENS2.2, WB_SENS2.3
- net SHORT_HW-: now also LONG_HW+.P$2, SHORT_HW-.P$1, TP25.TP, TP27.TP, WB_SENS1.1, WB_SENS1.6, WB_SENS1.8
- net WB_CURRENT+: now also POWER.2, WB_SENS2.7; no longer POWER.3, WB_SENS2.1
- net WB_CURRENT-: now also LONG_HW-.P$1, POWER.1, TP28.TP, WB_SENS1.5, WB_SENS2.3; no longer POWER.4, U1.OUTA, WB_SENS2.6
Other:
- note removed: "Linearisation of WB"
- note removed: "This will let node A see GND!"

Commit message: new traces
Parts:
- removed PT$0: PTS1206A, PTS1206:PTS1206A
- removed R4, R7: (no value), resistor:R-US_M0805
- removed TP1, TP10, TP12, TP14, TP16, TP18, TP2, TP20, TP22, TP24, TP25, TP26, TP27, TP28, TP3, TP4, TP6, TP8: TPTP10SQ, testpad:TPTP10SQ
- added POT_1, POT_2, POT_LONG_HW, POT_SHORT_HW: 67WR200LFR$1, POTENTIOMETER_67WR200LFR:67WR200LFR$1
- added PT$6: PTS1206A, PTS1206:PTS1206A
Connections:
- removed net PT0_S+: PT$0.S+, PT_SENS2.3, TP2.TP
- removed net PT0_S-: PT$0.S-, PT_SENS2.4, TP4.TP
- removed net PT1_S+: PT$1.S+, PT_SENS1.2, TP10.TP
- removed net PT1_S-: PT$1.S-, PT_SENS1.1, TP12.TP
- removed net PT2_S+: PT$2.S+, PT_SENS2.5, TP6.TP
- removed net PT2_S-: PT$2.S-, PT_SENS2.6, TP8.TP
- removed net PT3_S+: PT$3.S+, PT_SENS2.2, TP18.TP
- removed net PT3_S-: PT$3.S-, PT_SENS2.1, TP20.TP
- removed net PT4_S+: PT$4.S+, PT_SENS2.8, TP14.TP
- removed net PT4_S-: PT$4.S-, PT_SENS2.7, TP16.TP
- removed net PT5_S+: PT$5.S+, PT_SENS1.4, TP22.TP
- removed net PT5_S-: PT$5.S-, PT_SENS1.3, TP24.TP
- new net N$1: LONG_HW-.P$1, LONG_HW-.P$2, POT_LONG_HW.2
- new net N$2: PT$1.-, PT$2.+, PT_SENS2.2, PT_SENS2.3
- new net N$3: PT$2.-, PT$3.+, PT_SENS2.4, PT_SENS2.5
- new net N$4: PT$3.-, PT$4.+, PT_SENS2.6, PT_SENS2.7
- new net N$5: PT$4.-, PT$5.+, PT_SENS1.1, PT_SENS2.8
- new net N$6: PT$5.-, PT$6.+, PT_SENS1.2, PT_SENS1.3
- new net N$8: POT_SHORT_HW.1, SHORT_HW+.P$1, SHORT_HW+.P$2
- net NODE_B: now also POT_1.1, POT_2.2, WB_SENS1.1; no longer R4.1, R7.2, WB_SENS1.7
- net PT_CURRENT+: now also PT_SENS2.1; no longer PT$0.+, PT$0.-, PT$1.-, PT$2.+, PT$2.-, PT$3.+, PT$3.-, PT$4.+, PT$4.-, PT$5.+, TP1.TP
- net PT_CURRENT-: now also PT$6.-, PT_SENS1.4; no longer PT$5.-, TP3.TP
- net SHORT_HW+: now also POT_1.2, POT_SHORT_HW.2; no longer R4.2, SHORT_HW+.P$1, SHORT_HW+.P$2, TP26.TP, WB_SENS1.2
- net SHORT_HW-: now also WB_SENS1.2; no longer TP25.TP, TP27.TP, WB_SENS1.1, WB_SENS1.6, WB_SENS1.8
- net WB_CURRENT-: now also POT_2.1, POT_LONG_HW.1, POWER.5; no longer LONG_HW-.P$1, LONG_HW-.P$2, POWER.1, R7.1, TP28.TP, WB_SENS1.5
Other:
- note removed: "OP-AMP A INPUT"
- note removed: "PT Sensors"
- moved on the sheet: LONG_HW+, LONG_HW-, SHORT_HW+, SHORT_HW-

Commit message: finish routing pt sensors tomorrow
Other:
- note removed: "OP-AMP A OUTPUT"
Changed lines of the file:
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@@
 <plain>
 <text x="208.28" y="259.08" size="2.54" layer="91">WHEATSTONE BRIDGE</text>
-<text x="233.68" y="-38.1" size="1.4224" layer="97">OP-AMP A OUTPUT</text>
 <text x="180.34" y="86.36" size="1.6764" layer="97">NODE A</text>
 <text x="167.64" y="200.66" size="3.81" layer="97">*DASH LINES REPERSENT SENSE LINES*</text>
@@
 <junction x="223.52" y="-25.4"/>
 <label x="160.02" y="-25.4" size="1.778" layer="95" rot="R180" xref="yes"/>
-<label x="223.52" y="-27.94" size="1.778" layer="95" rot="R270" xref="yes"/>
 <wire x1="281.94" y1="10.16" x2="271.78" y2="10.16" width="0.1524" layer="91" style="shortdash"/>
 <pinref part="WB_SENS2" gate="G$1" pin="3"/>
@@
 <net name="N$1" class="0">
 <segment>
-<wire x1="182.88" y1="25.4" x2="182.88" y2="20.32" width="0.1524" layer="91" style="shortdash"/>
-<wire x1="182.88" y1="30.48" x2="182.88" y2="25.4" width="0.1524" layer="91"/>
 <pinref part="LONG_HW-" gate="G$1" pin="P$1"/>
 <pinref part="LONG_HW-" gate="G$1" pin="P$2"/>
 <wire x1="177.8" y1="30.48" x2="182.88" y2="30.48" width="0.1524" layer="91"/>
-<junction x="182.88" y="30.48"/>
 <pinref part="POT_LONG_HW" gate="G$1" pin="2"/>
 <wire x1="177.8" y1="30.48" x2="177.8" y2="12.7" width="0.1524" layer="91"/>
@@
 </segment>
 </net>
-<net name="N$8" class="0">
-<segment>
+<net name="N$7" class="0">
+<segment>
+<pinref part="SHORT_HW+" gate="G$1" pin="P$1"/>
 <pinref part="SHORT_HW+" gate="G$1" pin="P$2"/>
 <wire x1="182.88" y1="139.7" x2="182.88" y2="142.24" width="0.1524" layer="91"/>
-<junction x="182.88" y="142.24"/>
-<pinref part="SHORT_HW+" gate="G$1" pin="P$1"/>
-<wire x1="177.8" y1="142.24" x2="177.8" y2="139.7" width="0.1524" layer="91"/>
 <wire x1="177.8" y1="142.24" x2="182.88" y2="142.24" width="0.1524" layer="91"/>
-<wire x1="182.88" y1="142.24" x2="182.88" y2="144.78" width="0.1524" layer="91" style="shortdash"/>
-<wire x1="182.88" y1="144.78" x2="200.66" y2="144.78" width="0.1524" layer="91" style="shortdash"/>
-<wire x1="200.66" y1="144.78" x2="200.66" y2="132.08" width="0.1524" layer="91" style="shortdash"/>
-<wire x1="200.66" y1="132.08" x2="213.36" y2="132.08" width="0.1524" layer="91" style="shortdash"/>
 <pinref part="POT_SHORT_HW" gate="G$1" pin="1"/>
 <wire x1="177.8" y1="152.4" x2="177.8" y2="142.24" width="0.1524" layer="91"/>
 <junction x="177.8" y="142.24"/>
-</segment>
-</net>
+<wire x1="177.8" y1="142.24" x2="177.8" y2="139.7" width="0.1524" layer="91"/>
+</segment>
+</net>
