File: THW/Eagle/THW_Design/v1.2.0.sch (EAGLE design)
At the start: 20 parts

Commit message: 4-wire sense
Connections:
- net N$1: now also WB_SENS2.6
- net N$7: now also WB_SENS1.1, WB_SENS2.4; no longer WB_SENS2.6
- net NODE_B: now also POWER.5, WB_SENS1.5; no longer WB_SENS1.1, WB_SENS2.4
- net SHORT_HW+: now also POWER.6, WB_SENS1.8; no longer WB_SENS1.4, WB_SENS2.5
- net SHORT_HW-: now also WB_SENS1.6, WB_SENS2.7
- net WB_CURRENT+: now also WB_SENS1.7; no longer WB_SENS1.3
- net WB_CURRENT-: now also WB_SENS2.5; no longer WB_SENS2.7

Commit message: push
Connections:
- net N$1: now also WB_SENS2.7; no longer WB_SENS2.8
- net N$3: now also PT_SENS2.3, PT_SENS2.6; no longer PT_SENS2.4, PT_SENS2.5
- net N$4: now also PT_SENS2.5; no longer PT_SENS2.6
- net N$9: now also PT_SENS2.4; no longer PT_SENS2.3
- net SHORT_HW-: now also WB_SENS2.8; no longer WB_SENS2.7
Changed lines of the file:
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@@
 </segment>
 <segment>
-<pinref part="WB_SENS2" gate="G$1" pin="7"/>
-<wire x1="213.36" y1="236.22" x2="203.2" y2="236.22" width="0.1524" layer="91" style="shortdash"/>
-<label x="203.2" y="236.22" size="2.1844" layer="95" rot="R180" xref="yes"/>
+<pinref part="WB_SENS2" gate="G$1" pin="8"/>
+<wire x1="236.22" y1="236.22" x2="243.84" y2="236.22" width="0.1524" layer="91" style="shortdash"/>
+<label x="243.84" y="236.22" size="2.1844" layer="95" xref="yes"/>
 </segment>
 </net>
@@
 <pinref part="PT$3" gate="G$1" pin="+"/>
 <wire x1="144.78" y1="289.56" x2="165.1" y2="289.56" width="0.1524" layer="91"/>
-<wire x1="144.78" y1="289.56" x2="144.78" y2="309.88" width="0.1524" layer="91" style="shortdash"/>
-<wire x1="144.78" y1="309.88" x2="193.04" y2="309.88" width="0.1524" layer="91" style="shortdash"/>
+<wire x1="144.78" y1="289.56" x2="144.78" y2="330.2" width="0.1524" layer="91" style="shortdash"/>
 <junction x="144.78" y="289.56"/>
-<pinref part="PT_SENS2" gate="G$1" pin="4"/>
-<wire x1="193.04" y1="309.88" x2="193.04" y2="330.2" width="0.1524" layer="91" style="shortdash"/>
-<wire x1="193.04" y1="330.2" x2="172.72" y2="330.2" width="0.1524" layer="91" style="shortdash"/>
-<wire x1="165.1" y1="289.56" x2="165.1" y2="302.26" width="0.1524" layer="91" style="shortdash"/>
-<wire x1="165.1" y1="302.26" x2="149.86" y2="302.26" width="0.1524" layer="91" style="shortdash"/>
+<pinref part="PT_SENS2" gate="G$1" pin="3"/>
+<wire x1="144.78" y1="330.2" x2="149.86" y2="330.2" width="0.1524" layer="91" style="shortdash"/>
+<wire x1="165.1" y1="289.56" x2="165.1" y2="312.42" width="0.1524" layer="91" style="shortdash"/>
+<wire x1="165.1" y1="312.42" x2="185.42" y2="312.42" width="0.1524" layer="91" style="shortdash"/>
 <junction x="165.1" y="289.56"/>
-<wire x1="149.86" y1="302.26" x2="147.32" y2="302.26" width="0.1524" layer="91" style="shortdash"/>
-<wire x1="147.32" y1="302.26" x2="147.32" y2="335.28" width="0.1524" layer="91" style="shortdash"/>
-<pinref part="PT_SENS2" gate="G$1" pin="5"/>
-<wire x1="147.32" y1="335.28" x2="149.86" y2="335.28" width="0.1524" layer="91" style="shortdash"/>
+<pinref part="PT_SENS2" gate="G$1" pin="6"/>
+<wire x1="185.42" y1="312.42" x2="185.42" y2="335.28" width="0.1524" layer="91" style="shortdash"/>
+<wire x1="185.42" y1="335.28" x2="172.72" y2="335.28" width="0.1524" layer="91" style="shortdash"/>
 </segment>
 </net>
@@
 <pinref part="PT$4" gate="G$1" pin="+"/>
 <wire x1="190.5" y1="289.56" x2="210.82" y2="289.56" width="0.1524" layer="91"/>
-<pinref part="PT_SENS2" gate="G$1" pin="6"/>
-<wire x1="190.5" y1="289.56" x2="190.5" y2="335.28" width="0.1524" layer="91" style="shortdash"/>
-<wire x1="190.5" y1="335.28" x2="172.72" y2="335.28" width="0.1524" layer="91" style="shortdash"/>
-<junction x="190.5" y="289.56"/>
 <wire x1="210.82" y1="289.56" x2="210.82" y2="365.76" width="0.1524" layer="91" style="shortdash"/>
-<wire x1="210.82" y1="365.76" x2="152.4" y2="365.76" width="0.1524" layer="91" style="shortdash"/>
+<wire x1="210.82" y1="365.76" x2="149.86" y2="365.76" width="0.1524" layer="91" style="shortdash"/>
 <junction x="210.82" y="289.56"/>
 <pinref part="PT_SENS2" gate="G$1" pin="7"/>
-<wire x1="152.4" y1="365.76" x2="149.86" y2="365.76" width="0.1524" layer="91" style="shortdash"/>
 <wire x1="149.86" y1="365.76" x2="149.86" y2="340.36" width="0.1524" layer="91" style="shortdash"/>
+<wire x1="190.5" y1="289.56" x2="190.5" y2="299.72" width="0.1524" layer="91" style="shortdash"/>
+<wire x1="190.5" y1="299.72" x2="134.62" y2="299.72" width="0.1524" layer="91" style="shortdash"/>
+<junction x="190.5" y="289.56"/>
+<pinref part="PT_SENS2" gate="G$1" pin="5"/>
+<wire x1="134.62" y1="299.72" x2="134.62" y2="335.28" width="0.1524" layer="91" style="shortdash"/>
+<wire x1="134.62" y1="335.28" x2="149.86" y2="335.28" width="0.1524" layer="91" style="shortdash"/>
 </segment>
 </net>
@@
 </segment>
 <segment>
-<pinref part="WB_SENS2" gate="G$1" pin="8"/>
-<wire x1="236.22" y1="236.22" x2="243.84" y2="236.22" width="0.1524" layer="91" style="shortdash"/>
-<label x="243.84" y="236.22" size="2.1844" layer="95" xref="yes"/>
+<pinref part="WB_SENS2" gate="G$1" pin="7"/>
+<wire x1="213.36" y1="236.22" x2="203.2" y2="236.22" width="0.1524" layer="91" style="shortdash"/>
+<label x="203.2" y="236.22" size="2.1844" layer="95" rot="R180" xref="yes"/>
 </segment>
 </net>
@@
 <net name="N$9" class="0">
 <segment>
-<pinref part="PT_SENS2" gate="G$1" pin="3"/>
-<wire x1="119.38" y1="330.2" x2="149.86" y2="330.2" width="0.1524" layer="91" style="shortdash"/>
 <pinref part="PT$2" gate="G$1" pin="+"/>
-<wire x1="119.38" y1="289.56" x2="119.38" y2="330.2" width="0.1524" layer="91" style="shortdash"/>
+<wire x1="119.38" y1="289.56" x2="119.38" y2="307.34" width="0.1524" layer="91" style="shortdash"/>
 <junction x="119.38" y="289.56"/>
 <pinref part="PT$1" gate="G$1" pin="-"/>
@@
 <wire x1="106.68" y1="325.12" x2="149.86" y2="325.12" width="0.1524" layer="91" style="shortdash"/>
 <junction x="106.68" y="289.56"/>
-</segment>
-</net>
+<wire x1="119.38" y1="307.34" x2="180.34" y2="307.34" width="0.1524" layer="91" style="shortdash"/>
+<pinref part="PT_SENS2" gate="G$1" pin="4"/>
+<wire x1="180.34" y1="307.34" x2="180.34" y2="330.2" width="0.1524" layer="91" style="shortdash"/>
+<wire x1="180.34" y1="330.2" x2="172.72" y2="330.2" width="0.1524" layer="91" style="shortdash"/>
+</segment>
+</net>

Commit message: changes
Parts:
- removed POT_LONG_HW, POT_SHORT_HW: 67WR200LFR$1, POTENTIOMETER_67WR200LFR:67WR200LFR$1
- added PAD1, PAD2, PAD3: (no value), wirepad:2,15/1,0
- added POT_3, POT_4: 67WR200LFR$1, POTENTIOMETER_67WR200LFR:67WR200LFR$1
Connections:
- new net GND: POWER.S1, POWER.S2, PT_SENS1.S1, PT_SENS1.S2, PT_SENS2.S1, PT_SENS2.S2, WB_SENS1.S1, WB_SENS1.S2, WB_SENS2.S1, WB_SENS2.S2
- net N$1: now also PAD3.P, POT_2.2; no longer POT_LONG_HW.2
- net N$7: now also PAD2.P, POT_1.1; no longer POT_SHORT_HW.1
- net NODE_B: now also POT_3.1, POT_4.2; no longer POT_1.1, POT_2.2
- net SHORT_HW+: now also POT_3.2; no longer POT_SHORT_HW.2
- net SHORT_HW-: now also PAD1.P
- net WB_CURRENT-: now also POT_4.1; no longer POT_LONG_HW.1
Other:
- moved on the sheet: POT_1, POT_2
