File: THW/Eagle/THW_Design/v1.2.0.brd (EAGLE design)
At the start: 100 x 200 mm, 21 parts

Commit message: V1 THW DONE :)!
Routing:
- net SHORT_HW-: track 206.1 -> 3.08 mm
- net N$9: track 208.5 -> 214.8 mm
- net PT_CURRENT+: track 157.7 -> 162.4 mm
- net N$5: track 412.8 -> 415.7 mm
- net N$4: track 407.6 -> 410.5 mm
- net PT_CURRENT-: track 255.8 -> 258.7 mm
- net N$3: track 264.4 -> 265.9 mm
Other:
- outline, holes or cut-outs redrawn
- board text added: "ASAD MOHIUDDIN"
- board text added: "MARCUS BANNERMAN"
- board text added: "THW BOARD V1 BY:"

Commit message: 4-wire sense
Connections:
- net N$1: now also WB_SENS2.6
- net N$7: now also WB_SENS1.1, WB_SENS2.4; no longer WB_SENS2.6
- net NODE_B: now also POWER.5, WB_SENS1.5; no longer WB_SENS1.1, WB_SENS2.4
- net SHORT_HW+: now also POWER.6, WB_SENS1.8; no longer WB_SENS1.4, WB_SENS2.5
- net SHORT_HW-: now also WB_SENS1.6, WB_SENS2.7
- net WB_CURRENT+: now also WB_SENS1.7; no longer WB_SENS1.3
- net WB_CURRENT-: now also WB_SENS2.5; no longer WB_SENS2.7
Routing:
- net N$1: track 40.1 -> 238.0 mm, vias 3 -> 4
- net SHORT_HW-: track 3.08 -> 81.1 mm
- net N$7: track 57.9 -> 126.2 mm
- net NODE_B: track 51.5 -> 34.2 mm
- net SHORT_HW+: track 91.2 -> 84.6 mm
- net N$3: track 265.9 -> 270.5 mm, vias 2 -> 3
- net N$4: track 410.5 -> 414.5 mm, vias 3 -> 4
- net PT_CURRENT-: track 258.7 -> 255.8 mm
- net N$5: track 415.7 -> 417.4 mm
- net WB_CURRENT-: track 59.8 -> 58.2 mm
- net WB_CURRENT+: track 13.6 -> 12.0 mm

Commit message: push
Connections:
- net N$1: now also WB_SENS2.7; no longer WB_SENS2.8
- net N$3: now also PT_SENS2.3, PT_SENS2.6; no longer PT_SENS2.4, PT_SENS2.5
- net N$4: now also PT_SENS2.5; no longer PT_SENS2.6
- net N$9: now also PT_SENS2.4; no longer PT_SENS2.3
- net SHORT_HW-: now also WB_SENS2.8; no longer WB_SENS2.7
Routing:
- net N$1: track 238.0 -> 113.4 mm, vias 4 -> 3
- net SHORT_HW-: track 81.1 -> 205.7 mm
- net N$9: track 214.8 -> 225.1 mm, vias 3 -> 4
- net N$4: track 414.5 -> 406.2 mm, vias 4 -> 3
- net N$3: track 270.5 -> 267.7 mm
Other:
- outline, holes or cut-outs redrawn

Commit message: changes
Parts:
- removed POT_LONG_HW, POT_SHORT_HW: 67WR200LFR$1, POTENTIOMETER_67WR200LFR:67WR200LF
- added PAD1, PAD2, PAD3: (no value), wirepad:2,15/1,0
- added POT_3, POT_4: 67WR200LFR$1, POTENTIOMETER_67WR200LFR:67WR200LF
- moved POT_2 20.1 mm to (54.7, 155.7), turned to 90 degrees
- moved POT_1 4.98 mm to (44.4, 165.2), turned to 270 degrees
Connections:
- new net GND: POWER.S1, POWER.S2, PT_SENS1.S1, PT_SENS1.S2, PT_SENS2.S1, PT_SENS2.S2, WB_SENS1.S1, WB_SENS1.S2, WB_SENS2.S1, WB_SENS2.S2
- net N$1: now also PAD3.1, POT_2.P$2; no longer POT_LONG_HW.P$2
- net N$7: now also PAD2.1, POT_1.P$1; no longer POT_SHORT_HW.P$1
- net NODE_B: now also POT_3.P$1, POT_4.P$2; no longer POT_1.P$1, POT_2.P$2
- net SHORT_HW+: now also POT_3.P$2; no longer POT_SHORT_HW.P$2
- net SHORT_HW-: now also PAD1.1
- net WB_CURRENT-: now also POT_4.P$1; no longer POT_LONG_HW.P$1
Routing:
- net N$3: track 267.7 -> 268.7 mm
- net WB_CURRENT-: track 58.2 -> 57.5 mm
- net PT_CURRENT-: track 255.8 -> 255.1 mm
- net NODE_B: track 34.2 -> 33.6 mm
- net N$9: track 225.1 -> 225.7 mm
- added copper zone on layer 1, net GND
- removed copper zone on layer 1, net TSHEILD
Other:
- board text added: "LONG_HW"
- board text added: "LONG_HW_S"
- board text added: "POT_1"
- board text added: "POT_2"
- board text added: "POT_3"
- board text added: "POT_4"
- board text added: "PT_1"
- board text added: "PT_2"
- board text added: "PT_3"
- board text added: "PT_4"
- board text added: "PT_5"
- board text added: "PT_6"
- board text added: "PT_POWER"
- board text added: "R_CURRENT"
- board text added: "SHORT_HW"
- board text added: "SHORT_HW_S"
- board text added: "WB_NODE"
- board text added: "WB_POWER"
- board text added: "WB_SENS"
